Commit message: modifying gazebo xacro now

File: quad_simulator/go2_description/xacro/const.xacro (robot description, xacro)
@@ -19,4 +19,8 @@
     <xacro:property name="stick_radius" value="0.01"/>
     <xacro:property name="stick_length" value="0.2"/>
+    <xacro:property name="toe_friction" value="0.2"/>
+    <xacro:property name="toe_lateral_friction" value="0.2"/>
+    <xacro:property name="toe_stiffness" value="30000.0"/>
+    <xacro:property name="toe_damping" value="1000.0"/>
     <!-- kinematic value -->
     <xacro:property name="thigh_offset" value="0.0955"/>

File: quad_simulator/go2_description/xacro/leg.xacro (robot description, xacro)
@@ -2,6 +2,41 @@
 <robot xmlns:xacro="http://www.ros.org/wiki/xacro">
     <xacro:include filename="$(find go2_description)/xacro/transmission.xacro"/>
-    <xacro:macro name="leg" params="name mirror mirror_dae front_hind front_hind_dae">
-        <joint name="${name}_hip_joint" type="revolute">
+    <xacro:macro name="leg" params="suffix mirror mirror_dae front_hind front_hind_dae
+                                hipJointName kneeJointName abductionJointName *origin">
+        <link name="hip${suffix}">
+            <visual name="hip${suffix}_visual">
+                <xacro:if value="${(mirror_dae == True) and (front_hind_dae == True)}">
+                    <origin rpy="0 0 0" xyz="0 0 0"/>
+                </xacro:if>
+                <xacro:if value="${(mirror_dae == False) and (front_hind_dae == True)}">
+                    <origin rpy="${PI} 0 0" xyz="0 0 0"/>
+                </xacro:if>
+                <xacro:if value="${(mirror_dae == True) and (front_hind_dae == False)}">
+                    <origin rpy="0 ${PI} 0" xyz="0 0 0"/>
+                </xacro:if>
+                <xacro:if value="${(mirror_dae == False) and (front_hind_dae == False)}">
+                    <origin rpy="${PI} ${PI} 0" xyz="0 0 0"/>
+                </xacro:if>
+                <geometry>
+                    <mesh filename="package://go2_description/meshes/hip.dae" scale="1 1 1"/>
+                </geometry>
+                <!-- <material name="orange"/> -->
+            </visual>
+            <collision>
+                <origin rpy="${PI/2.0} 0 0" xyz="0 ${hip_offset*mirror} 0"/>
+                <geometry>
+                    <cylinder length="${hip_length}" radius="${hip_radius}"/>
+                </geometry>
+            </collision>
+            <inertial>
+                <origin rpy="0 0 0" xyz="${hip_com_x*front_hind} ${hip_com_y*mirror} ${hip_com_z}"/>
+                <mass value="${hip_mass}"/>
+                <inertia
+                    ixx="${hip_ixx}" ixy="${hip_ixy*mirror*front_hind}" ixz="${hip_ixz*front_hind}"
+                    iyy="${hip_iyy}" iyz="${hip_iyz*mirror}"
+                    izz="${hip_izz}"/>
+            </inertial>
+        </link>
+        <joint name="${abductionJointName}" type="revolute">
             <xacro:if value="${(mirror_dae == False) and (front_hind_dae == True)}">
                 <origin rpy="0 0 0" xyz="${leg_offset_x} ${-leg_offset_y} 0"/>
@@ -17,5 +52,5 @@
             </xacro:if>
             <parent link="trunk"/>
-            <child link="${name}_hip"/>
+            <child link="hip${suffix}"/>
             <axis xyz="1 0 0"/>
             <dynamics damping="${damping}" friction="${friction}"/>
@@ -27,48 +62,20 @@
             </xacro:if>
         </joint>
-        <link name="${name}_hip">
-            <visual>
-                <xacro:if value="${(mirror_dae == True) and (front_hind_dae == True)}">
-                    <origin rpy="0 0 0" xyz="0 0 0"/>
-                </xacro:if>
-                <xacro:if value="${(mirror_dae == False) and (front_hind_dae == True)}">
-                    <origin rpy="${PI} 0 0" xyz="0 0 0"/>
-                </xacro:if>
-                <xacro:if value="${(mirror_dae == True) and (front_hind_dae == False)}">
-                    <origin rpy="0 ${PI} 0" xyz="0 0 0"/>
-                </xacro:if>
-                <xacro:if value="${(mirror_dae == False) and (front_hind_dae == False)}">
-                    <origin rpy="${PI} ${PI} 0" xyz="0 0 0"/>
-                </xacro:if>
-                <geometry>
-                    <mesh filename="package://go2_description/meshes/hip.dae" scale="1 1 1"/>
-                </geometry>
-                <!-- <material name="orange"/> -->
-            </visual>
+        <!-- this link is only for collision -->
+        <link name="thigh_shoulder${suffix}">
             <collision>
-                <origin rpy="${PI/2.0} 0 0" xyz="0 ${hip_offset*mirror} 0"/>
-                <geometry>
-                    <cylinder length="${hip_length}" radius="${hip_radius}"/>
-                </geometry>
-            </collision>
-            <inertial>
-                <origin rpy="0 0 0" xyz="${hip_com_x*front_hind} ${hip_com_y*mirror} ${hip_com_z}"/>
-                <mass value="${hip_mass}"/>
-                <inertia
-                    ixx="${hip_ixx}" ixy="${hip_ixy*mirror*front_hind}" ixz="${hip_ixz*front_hind}"
-                    iyy="${hip_iyy}" iyz="${hip_iyz*mirror}"
-                    izz="${hip_izz}"/>
-            </inertial>
-        </link>
-        <joint name="${name}_thigh_joint" type="revolute">
-            <origin rpy="0 0 0" xyz="0 ${thigh_offset*mirror} 0"/>
-            <parent link="${name}_hip"/>
-            <child link="${name}_thigh"/>
-            <axis xyz="0 1 0"/>
-            <dynamics damping="${damping}" friction="${friction}"/>
-            <limit effort="${thigh_torque_max}" velocity="${thigh_velocity_max}" lower="${thigh_position_min}" upper="${thigh_position_max}"/>
-        </joint>
-        <link name="${name}_thigh">
-            <visual>
+                <origin rpy="${PI/2.0} 0 0" xyz="0 0 0"/>
+                <geometry>
+                    <cylinder length="${thigh_shoulder_length}" radius="${thigh_shoulder_radius}"/>
+                </geometry>
+            </collision>
+        </link>
+        <joint name="hip${suffix}_fixed" type="fixed">
+            <origin rpy="0 0 0" xyz="0 ${(thigh_shoulder_length/2.0+hip_offset)*mirror} 0"/>
+            <parent link="hip${suffix}"/>
+            <child link="thigh_shoulder${suffix}"/>
+        </joint>
+        <link name="upper${suffix}">
+            <visual name="upper${suffix}_visual">
                 <origin rpy="0 0 0" xyz="0 0 0"/>
                 <geometry>
@@ -82,5 +89,5 @@
                 <!-- <material name="orange"/> -->
             </visual>
-            <collision>
+            <collision name="upper${suffix}_collision">
                 <origin rpy="0 ${PI/2.0} 0" xyz="0 0 ${-thigh_length/2.0}"/>
                 <geometry>
@@ -97,42 +104,45 @@
             </inertial>
         </link>
-        <joint name="${name}_calf_joint" type="revolute">
+        <joint name="${hipJointName}" type="revolute">
+            <origin rpy="0 0 0" xyz="0 ${thigh_offset*mirror} 0"/>
+            <parent link="hip${suffix}"/>
+            <child link="upper${suffix}"/>
+            <axis xyz="0 1 0"/>
+            <dynamics damping="${damping}" friction="${friction}"/>
+            <limit effort="${thigh_torque_max}" velocity="${thigh_velocity_max}" lower="${thigh_position_min}" upper="${thigh_position_max}"/>
+        </joint>
+        <link name="lower${suffix}">
+            <visual name="lower${suffix}_visual">
+                <origin rpy="0 0 0" xyz="0 0 0"/>
+                <geometry>
+                    <mesh filename="package://go2_description/meshes/calf.dae" scale="1 1 1"/>
+                </geometry>
+                <!-- <material name="orange"/> -->
+            </visual>
+            <collision name="lower${suffix}_collision">
+                <origin rpy="0 ${PI/2.0} 0" xyz="0 0 ${-calf_length/2.0}"/>
+                <geometry>
+                    <box size="${calf_length} ${calf_width} ${calf_height}"/>
+                </geometry>
+            </collision>
+            <inertial>
+                <origin rpy="0 0 0" xyz="${calf_com_x} ${calf_com_y} ${calf_com_z}"/>
+                <mass value="${calf_mass}"/>
+                <inertia
+                    ixx="${calf_ixx}" ixy="${calf_ixy}" ixz="${calf_ixz}"
+                    iyy="${calf_iyy}" iyz="${calf_iyz}"
+                    izz="${calf_izz}"/>
+            </inertial>
+        </link>
+         <joint name="${kneeJointName}" type="revolute">
             <origin rpy="0 0 0" xyz="0 0 ${-thigh_length}"/>
-            <parent link="${name}_thigh"/>
-            <child link="${name}_calf"/>
+            <parent link="upper${suffix}"/>
+            <child link="lower${suffix}"/>
             <axis xyz="0 1 0"/>
             <dynamics damping="${damping}" friction="${friction}"/>
             <limit effort="${calf_torque_max}" velocity="${calf_velocity_max}" lower="${calf_position_min}" upper="${calf_position_max}"/>
         </joint>
-        <link name="${name}_calf">
-            <visual>
-                <origin rpy="0 0 0" xyz="0 0 0"/>
-                <geometry>
-                    <mesh filename="package://go2_description/meshes/calf.dae" scale="1 1 1"/>
-                </geometry>
-                <!-- <material name="orange"/> -->
-            </visual>
-            <collision>
-                <origin rpy="0 ${PI/2.0} 0" xyz="0 0 ${-calf_length/2.0}"/>
-                <geometry>
-                    <box size="${calf_length} ${calf_width} ${calf_height}"/>
-                </geometry>
-            </collision>
-            <inertial>
-                <origin rpy="0 0 0" xyz="${calf_com_x} ${calf_com_y} ${calf_com_z}"/>
-                <mass value="${calf_mass}"/>
-                <inertia
-                    ixx="${calf_ixx}" ixy="${calf_ixy}" ixz="${calf_ixz}"
-                    iyy="${calf_iyy}" iyz="${calf_iyz}"
-                    izz="${calf_izz}"/>
-            </inertial>
-        </link>
-        <joint name="${name}_foot_fixed" type="fixed">0
-            <origin rpy="0 0 0" xyz="0 0 ${-(calf_length)}"/>
-            <parent link="${name}_calf"/>
-            <child link="${name}_foot"/>
-        </joint>
-        <link name="${name}_foot">
-            <visual>
+        <link name="toe${suffix}">
+            <visual name="toe${suffix}_visual">
                 <origin rpy="0 0 0" xyz="0 0 0"/>
                 <geometry>
@@ -141,9 +151,37 @@
                 <!-- <material name="orange"/> -->
             </visual>
-            <collision>
+            <collision name="toe${suffix}_collision">
                 <origin rpy="0 0 0" xyz="0 0 0"/>
                 <geometry>
                     <sphere radius="${foot_radius}"/>
                 </geometry>
+                <surface>
+                <bounce>
+                    <restitution_coefficient>0</restitution_coefficient>
+                    <threshold>1e+06</threshold>
+                </bounce>
+                <friction>
+                    <ode>
+                        <mu>${toe_friction}</mu>
+                        <mu2>${toe_lateral_friction}</mu2>
+                    </ode>
+                    <bullet>
+                        <rolling_friction>0.3</rolling_friction>
+                        <friction2>50</friction2>
+                    </bullet>
+                </friction>
+                <contact>
+                    <ode>
+                        <kp>${toe_stiffness}</kp>
+                        <kd>${toe_damping}</kd>
+                    </ode>
+                    <bullet>
+                        <kp>${toe_stiffness}</kp>
+                        <kd>${toe_damping}</kd>
+                        <split_impulse>1</split_impulse>
+                        <split_impulse_penetration_threshold>-0.01</split_impulse_penetration_threshold>
+                    </bullet>
+                </contact>
+            </surface>
             </collision>
             <inertial>
@@ -155,5 +193,10 @@
             </inertial>
         </link>
-        <xacro:leg_transmission name="${name}"/>
+        <joint name="jtoe${suffix}" type="fixed">0
+            <origin rpy="0 0 0" xyz="0 0 ${-(calf_length)}"/>
+            <parent link="lower${suffix}"/>
+            <child link="toe${suffix}"/>
+        </joint>
+        <xacro:leg_transmission  hipJointName="${hipJointName}" kneeJointName="${kneeJointName}" abductionJointName="${abductionJointName}"/>
     </xacro:macro>
 </robot>

File: quad_simulator/go2_description/xacro/robot.xacro (robot description, xacro)
@@ -5,10 +5,9 @@
     <xacro:include filename="$(find go2_description)/xacro/materials.xacro"/>
     <xacro:include filename="$(find go2_description)/xacro/leg.xacro"/>
-    <!-- <xacro:include filename="$(find go2_description)/xacro/stairs.xacro"/> -->
     <xacro:include filename="$(find go2_description)/xacro/gazebo.xacro"/>
-    <!-- <xacro:include filename="$(find go2_gazebo)/launch/stairs.urdf.xacro"/> -->
-    <!-- <xacro:stairs stairs="15" xpos="0" ypos="0" zpos="0" /> -->
     <!-- Rotor related joint and link is only for demonstrate location. -->
     <!-- Actually, the rotor will rotate and the joint is not fixed. Reduction ratio should be considered. -->
+    <!-- Rollover Protection mode will add an additional stick on the top, use "true" or "false" to switch it. -->
+    <xacro:property name="rolloverProtection" value="false"/>
     <!-- Debug mode will hung up the robot, use "true" or "false" to switch it. -->
     <xacro:if value="$(arg DEBUG)">
@@ -17,8 +16,8 @@
             <origin rpy="0 0 0" xyz="0 0 0"/>
             <parent link="world"/>
-            <child link="base"/>
+            <child link="body"/>
         </joint>
     </xacro:if>
-    <link name="base">
+    <link name="body">
         <visual>
             <origin rpy="0 0 0" xyz="0 0 0"/>
@@ -30,9 +29,9 @@
     <joint name="floating_base" type="fixed">
         <origin rpy="0 0 0" xyz="0 0 0"/>
-        <parent link="base"/>
+        <parent link="body"/>
         <child link="trunk"/>
     </joint>
     <link name="trunk">
-        <visual>
+        <visual name="body_visual">
             <origin rpy="0 0 0" xyz="0 0 0"/>
             <geometry>
@@ -41,5 +40,5 @@
             <!-- <material name="orange"/> -->
         </visual>
-        <collision>
+        <collision name="body_collision">
             <origin rpy="0 0 0" xyz="0 0 0"/>
             <geometry>
@@ -56,4 +55,33 @@
         </inertial>
     </link>
+    <xacro:if value="${(rolloverProtection == 'true')}">
+        <joint name="stick_joint" type="fixed">
+            <parent link="trunk"/>
+            <child link="stick_link"/>
+            <origin rpy="0 0 0" xyz="${0.18} 0 ${stick_length/2.0+0.08}"/>
+        </joint>
+        <link name="stick_link">
+            <visual>
+                <geometry>
+                    <cylinder length="${stick_length}" radius="${stick_radius}"/>
+                </geometry>
+                <origin rpy="0 0 0" xyz="0 0 0"/>
+                <material name="white"/>
+            </visual>
+            <collision>
+                <geometry>
+                    <cylinder length="${stick_length}" radius="${stick_radius}"/>
+                </geometry>
+                <origin rpy="0 0 0" xyz="0 0 0"/>
+            </collision>
+            <inertial>
+                <mass value="${stick_mass}"/>
+                <inertia
+                    ixx="${stick_mass / 2.0 * (stick_radius*stick_radius)}" ixy="0.0" ixz="0.0"
+                    iyy="${stick_mass / 12.0 * (3*stick_radius*stick_radius + stick_length*stick_length)}" iyz="0.0"
+                    izz="${stick_mass / 12.0 * (3*stick_radius*stick_radius + stick_length*stick_length)}"/>
+            </inertial>
+        </link>
+    </xacro:if>
     <joint name="imu_joint" type="fixed">
         <parent link="trunk"/>
@@ -81,33 +109,23 @@
         </collision>
     </link>
-    <!--
-    <joint name="load_joint" type="fixed">
-        <parent link="trunk"/>
-        <child link="load_link"/>
-        <origin rpy="0 0 0" xyz="0 0 0"/>
-    </joint>
-    <link name="load_link">
-        <inertial>
-            <mass value="5"/>
-            <origin rpy="0 0 0" xyz="0 0 0"/>
-            <inertia ixx="0.01" ixy="0" ixz="0" iyy="0.01" iyz="0" izz="0.01"/>
-        </inertial>
-        <visual>
-            <origin rpy="0 0 0" xyz="0 0 0.2"/>
-            <geometry>
-                <box size="0.5 0.3 0.2"/>
-            </geometry>
-        </visual>
-        <collision>
-            <origin rpy="0 0 0" xyz="0 0 0"/>
-            <geometry>
-                <box size=".001 .001 .001"/>
-            </geometry>
-        </collision>
-    </link>
--->
-    <xacro:leg name="FR" mirror="-1" mirror_dae= "False" front_hind="1"  front_hind_dae="True"  />
-    <xacro:leg name="FL" mirror="1"  mirror_dae="True"   front_hind="1"  front_hind_dae="True"  />
-    <xacro:leg name="RR" mirror="-1" mirror_dae="False"  front_hind="-1" front_hind_dae="False" />
-    <xacro:leg name="RL" mirror="1"  mirror_dae="True"   front_hind="-1" front_hind_dae="False" />
+        <!--FL-->
+    <xacro:leg suffix="0" mirror="1" mirror_dae="True" front_hind="1" front_hind_dae="True"
+               hipJointName="0" kneeJointName="1" abductionJointName="8">
+        <origin rpy="0 0 0" xyz="${leg_offset_x} ${leg_offset_y} 0"/>
+    </xacro:leg>
+    <!--RL-->
+    <xacro:leg suffix="1" mirror="1" mirror_dae="True" front_hind="-1" front_hind_dae="False"
+               hipJointName="2" kneeJointName="3" abductionJointName="9">
+        <origin rpy="0 0 0" xyz="${-leg_offset_x} ${leg_offset_y} 0"/>
+    </xacro:leg>
+    <!--FR-->
+    <xacro:leg suffix="2" mirror="-1" mirror_dae="False" front_hind="1" front_hind_dae="True"
+               hipJointName="4" kneeJointName="5" abductionJointName="10">
+        <origin rpy="0 0 0" xyz="${leg_offset_x} ${-leg_offset_y} 0"/>
+    </xacro:leg>
+    <!--RR-->
+    <xacro:leg suffix="3" mirror="-1" mirror_dae="False" front_hind="-1" front_hind_dae="False"
+               hipJointName="6" kneeJointName="7" abductionJointName="11">
+        <origin rpy="0 0 0" xyz="${-leg_offset_x} ${-leg_offset_y} 0"/>
+    </xacro:leg>
 </robot>

File: quad_simulator/go2_description/xacro/transmission.xacro (robot description, xacro)
@@ -1,35 +1,35 @@
 <?xml version="1.0"?>
 <robot xmlns:xacro="http://www.ros.org/wiki/xacro">
-    <xacro:macro name="leg_transmission" params="name">
-        <transmission name="${name}_hip_tran">
-            <type>transmission_interface/SimpleTransmission</type>
-            <joint name="${name}_hip_joint">
-            <hardwareInterface>hardware_interface/EffortJointInterface</hardwareInterface>
-            </joint>
-            <actuator name="${name}_hip_motor">
-            <hardwareInterface>hardware_interface/EffortJointInterface</hardwareInterface>
-            <mechanicalReduction>1</mechanicalReduction>
-            </actuator>
-        </transmission>
-        <transmission name="${name}_thigh_tran">
-            <type>transmission_interface/SimpleTransmission</type>
-            <joint name="${name}_thigh_joint">
-            <hardwareInterface>hardware_interface/EffortJointInterface</hardwareInterface>
-            </joint>
-            <actuator name="${name}_thigh_motor">
-            <hardwareInterface>hardware_interface/EffortJointInterface</hardwareInterface>
-            <mechanicalReduction>1</mechanicalReduction>
-            </actuator>
-        </transmission>
-        <transmission name="${name}_calf_tran">
-            <type>transmission_interface/SimpleTransmission</type>
-            <joint name="${name}_calf_joint">
-            <hardwareInterface>hardware_interface/EffortJointInterface</hardwareInterface>
-            </joint>
-            <actuator name="${name}_calf_motor">
-            <hardwareInterface>hardware_interface/EffortJointInterface</hardwareInterface>
-            <mechanicalReduction>1</mechanicalReduction>
-            </actuator>
-        </transmission>
+    <xacro:macro name="leg_transmission" params="hipJointName kneeJointName abductionJointName">
+        <transmission name="transmission_${abductionJointName}">
+    		<type>transmission_interface/SimpleTransmission</type>
+    		<joint name="${abductionJointName}">
+      			<hardwareInterface>hardware_interface/EffortJointInterface</hardwareInterface>
+    		</joint>
+    		<actuator name="motor_${abductionJointName}">
+      			<hardwareInterface>EffortJointInterface</hardwareInterface>
+      			<mechanicalReduction>1</mechanicalReduction>
+    		</actuator>
+  		</transmission>
+        <transmission name="transmission_${hipJointName}">
+    		<type>transmission_interface/SimpleTransmission</type>
+    		<joint name="${hipJointName}">
+      			<hardwareInterface>hardware_interface/EffortJointInterface</hardwareInterface>
+    		</joint>
+    		<actuator name="motor_${hipJointName}">
+      			<hardwareInterface>EffortJointInterface</hardwareInterface>
+      			<mechanicalReduction>1</mechanicalReduction>
+    		</actuator>
+  		</transmission>
+        <transmission name="transmission_${kneeJointName}">
+    		<type>transmission_interface/SimpleTransmission</type>
+    		<joint name="${kneeJointName}">
+      			<hardwareInterface>hardware_interface/EffortJointInterface</hardwareInterface>
+    		</joint>
+    		<actuator name="motor_${kneeJointName}">
+      			<hardwareInterface>EffortJointInterface</hardwareInterface>
+      			<mechanicalReduction>1</mechanicalReduction>
+    		</actuator>
+  		</transmission>
     </xacro:macro>
 </robot>
