Commit message: re-generated sdf and urdf

File: quad_simulator/go2_description/urdf/go2.urdf (robot description, URDF)
Before this commit: robot go2_description, 29 links, 28 joints
Links:
- removed link FL_calflower
- removed link FL_calflower1
- removed link FR_calflower
- removed link FR_calflower1
- removed link Head_lower
- removed link Head_upper
- removed link RL_calflower
- removed link RL_calflower1
- removed link RR_calflower
- removed link RR_calflower1
- removed link imu
- removed link radar
- added link imu_link, mass 0.001; collision box size=.001 .001 .001; visual box size=0.001 0.001 0.001
- added link trunk, mass 6.921; collision box size=0.3762 0.0935 0.114; visual mesh filename=package://go2_description/meshes/trunk.dae scale=1 1 1
- link FL_calf: geometry collision box size=0.213 0.016 0.016; visual mesh filename=package://go2_description/meshes/calf.dae scale=1 1 1
- link FL_foot: mass 0.04 -> 0.06; geometry collision sphere radius=0.02; visual sphere radius=0.01
- link FL_hip: geometry collision cylinder length=0.04 radius=0.046; visual mesh filename=package://go2_description/meshes/hip.dae scale=1 1 1
- link FL_thigh: geometry collision box size=0.213 0.0245 0.034; visual mesh filename=package://go2_description/meshes/thigh.dae scale=1 1 1
- link FR_calf: geometry collision box size=0.213 0.016 0.016; visual mesh filename=package://go2_description/meshes/calf.dae scale=1 1 1
- link FR_foot: mass 0.04 -> 0.06; geometry collision sphere radius=0.02; visual sphere radius=0.01
- link FR_hip: geometry collision cylinder length=0.04 radius=0.046; visual mesh filename=package://go2_description/meshes/hip.dae scale=1 1 1
- link FR_thigh: geometry collision box size=0.213 0.0245 0.034; visual mesh filename=package://go2_description/meshes/thigh_mirror.dae scale=1 1 1
- link RL_calf: geometry collision box size=0.213 0.016 0.016; visual mesh filename=package://go2_description/meshes/calf.dae scale=1 1 1
- link RL_foot: mass 0.04 -> 0.06; geometry collision sphere radius=0.02; visual sphere radius=0.01
- link RL_hip: geometry collision cylinder length=0.04 radius=0.046; visual mesh filename=package://go2_description/meshes/hip.dae scale=1 1 1
- link RL_thigh: geometry collision box size=0.213 0.0245 0.034; visual mesh filename=package://go2_description/meshes/thigh.dae scale=1 1 1
- link RR_calf: geometry collision box size=0.213 0.016 0.016; visual mesh filename=package://go2_description/meshes/calf.dae scale=1 1 1
- link RR_foot: mass 0.04 -> 0.06; geometry collision sphere radius=0.02; visual sphere radius=0.01
- link RR_hip: geometry collision cylinder length=0.04 radius=0.046; visual mesh filename=package://go2_description/meshes/hip.dae scale=1 1 1
- link RR_thigh: geometry collision box size=0.213 0.0245 0.034; visual mesh filename=package://go2_description/meshes/thigh_mirror.dae scale=1 1 1
- link base: mass 6.921 -> None; geometry visual box size=0.001 0.001 0.001
Joints:
- removed joint FL_calflower1_joint
- removed joint FL_calflower_joint
- removed joint FL_foot_joint
- removed joint FR_calflower1_joint
- removed joint FR_calflower_joint
- removed joint FR_foot_joint
- removed joint Head_lower_joint
- removed joint Head_upper_joint
- removed joint RL_calflower1_joint
- removed joint RL_calflower_joint
- removed joint RL_foot_joint
- removed joint RR_calflower1_joint
- removed joint RR_calflower_joint
- removed joint RR_foot_joint
- removed joint radar_joint
- added joint FL_foot_fixed: type fixed, parent FL_calf, child FL_foot, origin xyz=0 0 -0.213 rpy=0 0 0
- added joint FR_foot_fixed: type fixed, parent FR_calf, child FR_foot, origin xyz=0 0 -0.213 rpy=0 0 0
- added joint RL_foot_fixed: type fixed, parent RL_calf, child RL_foot, origin xyz=0 0 -0.213 rpy=0 0 0
- added joint RR_foot_fixed: type fixed, parent RR_calf, child RR_foot, origin xyz=0 0 -0.213 rpy=0 0 0
- added joint floating_base: type fixed, parent base, child trunk, origin xyz=0 0 0 rpy=0 0 0
- joint FL_calf_joint: limit lower=-2.7227 upper=-0.83776 effort=45.43 velocity=15.70 -> lower=-2.7227 upper=-0.83776 effort=35.55 velocity=20.06
- joint FL_hip_joint: parent base -> trunk
- joint FR_calf_joint: limit lower=-2.7227 upper=-0.83776 effort=45.43 velocity=15.70 -> lower=-2.7227 upper=-0.83776 effort=35.55 velocity=20.06
- joint FR_hip_joint: parent base -> trunk
- joint RL_calf_joint: limit lower=-2.7227 upper=-0.83776 effort=45.43 velocity=15.70 -> lower=-2.7227 upper=-0.83776 effort=35.55 velocity=20.06
- joint RL_hip_joint: parent base -> trunk
- joint RL_thigh_joint: limit lower=-0.5236 upper=4.5379 effort=23.7 velocity=30.1 -> lower=-1.5708 upper=3.4907 effort=23.7 velocity=30.1
- joint RR_calf_joint: limit lower=-2.7227 upper=-0.83776 effort=45.43 velocity=15.70 -> lower=-2.7227 upper=-0.83776 effort=35.55 velocity=20.06
- joint RR_hip_joint: parent base -> trunk
- joint RR_thigh_joint: limit lower=-0.5236 upper=4.5379 effort=23.7 velocity=30.1 -> lower=-1.5708 upper=3.4907 effort=23.7 velocity=30.1
- joint imu_joint: axis 0 0 0 -> (none); child imu -> imu_link; origin xyz=-0.02557 0 0.04232 rpy=0 0 0 -> xyz=0 0 0 rpy=0 0 0; parent base -> trunk

Commit message: only getting robot driver error now, robot material not showing on rviz

File: quad_simulator/go2_description/urdf/go2.urdf (robot description, URDF)
Before this commit: robot go2, 19 links, 18 joints
Links:
- removed link imu_link
- removed link trunk
- added link FL_calflower; collision cylinder length=0.065 radius=0.011
- added link FL_calflower1; collision cylinder length=0.03 radius=0.0155
- added link FR_calflower; collision cylinder length=0.065 radius=0.011
- added link FR_calflower1; collision cylinder length=0.03 radius=0.0155
- added link Head_lower, mass 0.001; collision sphere radius=0.047
- added link Head_upper, mass 0.001; collision cylinder length=0.09 radius=0.05
- added link RL_calflower; collision cylinder length=0.065 radius=0.011
- added link RL_calflower1; collision cylinder length=0.03 radius=0.0155
- added link RR_calflower; collision cylinder length=0.065 radius=0.011
- added link RR_calflower1; collision cylinder length=0.03 radius=0.0155
- added link imu, mass 0
- added link radar, mass 0
- link FL_calf: geometry collision cylinder length=0.12 radius=0.012; visual mesh filename=package://go2_description/dae/calf.dae
- link FL_foot: mass 0.06 -> 0.04; geometry collision sphere radius=0.022; visual mesh filename=package://go2_description/dae/foot.dae
- link FL_hip: geometry collision cylinder length=0.04 radius=0.046; visual mesh filename=package://go2_description/dae/hip.dae
- link FL_thigh: geometry collision box size=0.213 0.0245 0.034; visual mesh filename=package://go2_description/dae/thigh.dae
- link FR_calf: geometry collision cylinder length=0.12 radius=0.013; visual mesh filename=package://go2_description/dae/calf_mirror.dae
- link FR_foot: mass 0.06 -> 0.04; geometry collision sphere radius=0.022; visual mesh filename=package://go2_description/dae/foot.dae
- link FR_hip: geometry collision cylinder length=0.04 radius=0.046; visual mesh filename=package://go2_description/dae/hip.dae
- link FR_thigh: geometry collision box size=0.213 0.0245 0.034; visual mesh filename=package://go2_description/dae/thigh_mirror.dae
- link RL_calf: geometry collision cylinder length=0.12 radius=0.013; visual mesh filename=package://go2_description/dae/calf.dae
- link RL_foot: mass 0.06 -> 0.04; geometry collision sphere radius=0.022; visual mesh filename=package://go2_description/dae/foot.dae
- link RL_hip: geometry collision cylinder length=0.04 radius=0.046; visual mesh filename=package://go2_description/dae/hip.dae
- link RL_thigh: geometry collision box size=0.213 0.0245 0.034; visual mesh filename=package://go2_description/dae/thigh.dae
- link RR_calf: geometry collision cylinder length=0.12 radius=0.013; visual mesh filename=package://go2_description/dae/calf_mirror.dae
- link RR_foot: mass 0.06 -> 0.04; geometry collision sphere radius=0.022; visual mesh filename=package://go2_description/dae/foot.dae
- link RR_hip: geometry collision cylinder length=0.04 radius=0.046; visual mesh filename=package://go2_description/dae/hip.dae
- link RR_thigh: geometry collision box size=0.213 0.0245 0.034; visual mesh filename=package://go2_description/dae/thigh_mirror.dae
- link base: mass None -> 6.921; geometry collision box size=0.3762 0.0935 0.114; visual mesh filename=package://go2_description/dae/base.dae
Joints:
- removed joint FL_foot_fixed
- removed joint FR_foot_fixed
- removed joint RL_foot_fixed
- removed joint RR_foot_fixed
- removed joint floating_base
- added joint FL_calflower1_joint: type fixed, parent FL_calflower, child FL_calflower1, origin xyz=-0.01 0 -0.04 rpy=0 0.48 0, axis 0 0 0
- added joint FL_calflower_joint: type fixed, parent FL_calf, child FL_calflower, origin xyz=0.020 0 -0.148 rpy=0 0.05 0, axis 0 0 0
- added joint FL_foot_joint: type fixed, parent FL_calf, child FL_foot, origin xyz=0 0 -0.213 rpy=0 0 0, axis 0 0 0
- added joint FR_calflower1_joint: type fixed, parent FR_calflower, child FR_calflower1, origin xyz=-0.01 0 -0.04 rpy=0 0.48 0, axis 0 0 0
- added joint FR_calflower_joint: type fixed, parent FR_calf, child FR_calflower, origin xyz=0.020 0 -0.148 rpy=0 0.05 0, axis 0 0 0
- added joint FR_foot_joint: type fixed, parent FR_calf, child FR_foot, origin xyz=0 0 -0.213 rpy=0 0 0, axis 0 0 0
- added joint Head_lower_joint: type fixed, parent Head_upper, child Head_lower, origin xyz=0.008 0 -0.07 rpy=0 0 0, axis 0 0 0
- added joint Head_upper_joint: type fixed, parent base, child Head_upper, origin xyz=0.285 0 0.01 rpy=0 0 0, axis 0 0 0
- added joint RL_calflower1_joint: type fixed, parent RL_calflower, child RL_calflower1, origin xyz=-0.01 0 -0.04 rpy=0 0.48 0, axis 0 0 0
- added joint RL_calflower_joint: type fixed, parent RL_calf, child RL_calflower, origin xyz=0.020 0 -0.148 rpy=0 0.05 0, axis 0 0 0
- added joint RL_foot_joint: type fixed, parent RL_calf, child RL_foot, origin xyz=0 0 -0.213 rpy=0 0 0, axis 0 0 0
- added joint RR_calflower1_joint: type fixed, parent RR_calflower, child RR_calflower1, origin xyz=-0.01 0 -0.04 rpy=0 0.48 0, axis 0 0 0
- added joint RR_calflower_joint: type fixed, parent RR_calf, child RR_calflower, origin xyz=0.020 0 -0.148 rpy=0 0.05 0, axis 0 0 0
- added joint RR_foot_joint: type fixed, parent RR_calf, child RR_foot, origin xyz=0 0 -0.213 rpy=0 0 0, axis 0 0 0
- added joint radar_joint: type fixed, parent base, child radar, origin xyz=0.28945 0 -0.046825 rpy=0 2.8782 0, axis 0 0 0
- joint FL_calf_joint: limit lower=-2.7227 upper=-0.83776 effort=35.55 velocity=20.06 -> lower=-2.7227 upper=-0.83776 effort=45.43 velocity=15.70
- joint FL_hip_joint: parent trunk -> base
- joint FR_calf_joint: limit lower=-2.7227 upper=-0.83776 effort=35.55 velocity=20.06 -> lower=-2.7227 upper=-0.83776 effort=45.43 velocity=15.70
- joint FR_hip_joint: parent trunk -> base
- joint RL_calf_joint: limit lower=-2.7227 upper=-0.83776 effort=35.55 velocity=20.06 -> lower=-2.7227 upper=-0.83776 effort=45.43 velocity=15.70
- joint RL_hip_joint: parent trunk -> base
- joint RL_thigh_joint: limit lower=-1.5708 upper=3.4907 effort=23.7 velocity=30.1 -> lower=-0.5236 upper=4.5379 effort=23.7 velocity=30.1
- joint RR_calf_joint: limit lower=-2.7227 upper=-0.83776 effort=35.55 velocity=20.06 -> lower=-2.7227 upper=-0.83776 effort=45.43 velocity=15.70
- joint RR_hip_joint: parent trunk -> base
- joint RR_thigh_joint: limit lower=-1.5708 upper=3.4907 effort=23.7 velocity=30.1 -> lower=-0.5236 upper=4.5379 effort=23.7 velocity=30.1
- joint imu_joint: axis (none) -> 0 0 0; child imu_link -> imu; origin xyz=0 0 0 rpy=0 0 0 -> xyz=-0.02557 0 0.04232 rpy=0 0 0; parent trunk -> base

Commit message: need to rename every link in the urdf according to naming convention, then change sdf file also

File: quad_simulator/go2_description/urdf/go2.urdf (robot description, URDF)
Before this commit: robot go2_description, 29 links, 28 joints
Links:
- removed link base
- added link body, mass 6.921; collision box size=0.3762 0.0935 0.114; visual mesh filename=package://go2_description/dae/body.dae
Joints:
- joint FL_hip_joint: parent base -> body
- joint FR_hip_joint: parent base -> body
- joint Head_upper_joint: parent base -> body
- joint RL_hip_joint: parent base -> body
- joint RR_hip_joint: parent base -> body
- joint imu_joint: parent base -> body
- joint radar_joint: parent base -> body

Commit message: created new urdf and sdf files

File: quad_simulator/go2_description/urdf/go2.urdf (robot description, URDF)
Before this commit: robot go2, 19 links, 18 joints
Links:
- removed link FL_calf
- removed link FL_foot
- removed link FL_hip
- removed link FL_thigh
- removed link FR_calf
- removed link FR_foot
- removed link FR_hip
- removed link FR_thigh
- removed link RL_calf
- removed link RL_foot
- removed link RL_hip
- removed link RL_thigh
- removed link RR_calf
- removed link RR_foot
- removed link RR_hip
- removed link RR_thigh
- removed link base
- added link body; visual box size=0.001 0.001 0.001
- added link hip0, mass 0.678; collision cylinder length=0.04 radius=0.046; visual mesh filename=package://go2_description/meshes/hip.dae scale=1 1 1
- added link hip1, mass 0.678; collision cylinder length=0.04 radius=0.046; visual mesh filename=package://go2_description/meshes/hip.dae scale=1 1 1
- added link hip2, mass 0.678; collision cylinder length=0.04 radius=0.046; visual mesh filename=package://go2_description/meshes/hip.dae scale=1 1 1
- added link hip3, mass 0.678; collision cylinder length=0.04 radius=0.046; visual mesh filename=package://go2_description/meshes/hip.dae scale=1 1 1
- added link lower0, mass 0.154; collision box size=0.213 0.016 0.016; visual mesh filename=package://go2_description/meshes/calf.dae scale=1 1 1
- added link lower1, mass 0.154; collision box size=0.213 0.016 0.016; visual mesh filename=package://go2_description/meshes/calf.dae scale=1 1 1
- added link lower2, mass 0.154; collision box size=0.213 0.016 0.016; visual mesh filename=package://go2_description/meshes/calf.dae scale=1 1 1
- added link lower3, mass 0.154; collision box size=0.213 0.016 0.016; visual mesh filename=package://go2_description/meshes/calf.dae scale=1 1 1
- added link thigh_shoulder0; collision cylinder length=0.032 radius=0.041
- added link thigh_shoulder1; collision cylinder length=0.032 radius=0.041
- added link thigh_shoulder2; collision cylinder length=0.032 radius=0.041
- added link thigh_shoulder3; collision cylinder length=0.032 radius=0.041
- added link toe0, mass 0.06; collision sphere radius=0.02; visual sphere radius=0.01
- added link toe1, mass 0.06; collision sphere radius=0.02; visual sphere radius=0.01
- added link toe2, mass 0.06; collision sphere radius=0.02; visual sphere radius=0.01
- added link toe3, mass 0.06; collision sphere radius=0.02; visual sphere radius=0.01
- added link upper0, mass 1.152; collision box size=0.213 0.0245 0.034; visual mesh filename=package://go2_description/meshes/thigh.dae scale=1 1 1
- added link upper1, mass 1.152; collision box size=0.213 0.0245 0.034; visual mesh filename=package://go2_description/meshes/thigh.dae scale=1 1 1
- added link upper2, mass 1.152; collision box size=0.213 0.0245 0.034; visual mesh filename=package://go2_description/meshes/thigh_mirror.dae scale=1 1 1
- added link upper3, mass 1.152; collision box size=0.213 0.0245 0.034; visual mesh filename=package://go2_description/meshes/thigh_mirror.dae scale=1 1 1
Joints:
- removed joint FL_calf_joint
- removed joint FL_foot_fixed
- removed joint FL_hip_joint
- removed joint FL_thigh_joint
- removed joint FR_calf_joint
- removed joint FR_foot_fixed
- removed joint FR_hip_joint
- removed joint FR_thigh_joint
- removed joint RL_calf_joint
- removed joint RL_foot_fixed
- removed joint RL_hip_joint
- removed joint RL_thigh_joint
- removed joint RR_calf_joint
- removed joint RR_foot_fixed
- removed joint RR_hip_joint
- removed joint RR_thigh_joint
- added joint 0: type revolute, parent hip0, child upper0, origin xyz=0 0.0955 0 rpy=0 0 0, axis 0 1 0, limit lower=-1.5708 upper=3.4907 effort=23.7 velocity=30.1
- added joint 1: type revolute, parent upper0, child lower0, origin xyz=0 0 -0.213 rpy=0 0 0, axis 0 1 0, limit lower=-2.7227 upper=-0.83776 effort=35.55 velocity=20.06
- added joint 10: type revolute, parent trunk, child hip2, origin xyz=0.1934 -0.0465 0 rpy=0 0 0, axis 1 0 0, limit lower=-1.0472 upper=1.0472 effort=23.7 velocity=30.1
- added joint 11: type revolute, parent trunk, child hip3, origin xyz=-0.1934 -0.0465 0 rpy=0 0 0, axis 1 0 0, limit lower=-1.0472 upper=1.0472 effort=23.7 velocity=30.1
- added joint 2: type revolute, parent hip1, child upper1, origin xyz=0 0.0955 0 rpy=0 0 0, axis 0 1 0, limit lower=-1.5708 upper=3.4907 effort=23.7 velocity=30.1
- added joint 3: type revolute, parent upper1, child lower1, origin xyz=0 0 -0.213 rpy=0 0 0, axis 0 1 0, limit lower=-2.7227 upper=-0.83776 effort=35.55 velocity=20.06
- added joint 4: type revolute, parent hip2, child upper2, origin xyz=0 -0.0955 0 rpy=0 0 0, axis 0 1 0, limit lower=-1.5708 upper=3.4907 effort=23.7 velocity=30.1
- added joint 5: type revolute, parent upper2, child lower2, origin xyz=0 0 -0.213 rpy=0 0 0, axis 0 1 0, limit lower=-2.7227 upper=-0.83776 effort=35.55 velocity=20.06
- added joint 6: type revolute, parent hip3, child upper3, origin xyz=0 -0.0955 0 rpy=0 0 0, axis 0 1 0, limit lower=-1.5708 upper=3.4907 effort=23.7 velocity=30.1
- added joint 7: type revolute, parent upper3, child lower3, origin xyz=0 0 -0.213 rpy=0 0 0, axis 0 1 0, limit lower=-2.7227 upper=-0.83776 effort=35.55 velocity=20.06
- added joint 8: type revolute, parent trunk, child hip0, origin xyz=0.1934 0.0465 0 rpy=0 0 0, axis 1 0 0, limit lower=-1.0472 upper=1.0472 effort=23.7 velocity=30.1
- added joint 9: type revolute, parent trunk, child hip1, origin xyz=-0.1934 0.0465 0 rpy=0 0 0, axis 1 0 0, limit lower=-1.0472 upper=1.0472 effort=23.7 velocity=30.1
- added joint hip0_fixed: type fixed, parent hip0, child thigh_shoulder0, origin xyz=0 0.1115 0 rpy=0 0 0
- added joint hip1_fixed: type fixed, parent hip1, child thigh_shoulder1, origin xyz=0 0.1115 0 rpy=0 0 0
- added joint hip2_fixed: type fixed, parent hip2, child thigh_shoulder2, origin xyz=0 -0.1115 0 rpy=0 0 0
- added joint hip3_fixed: type fixed, parent hip3, child thigh_shoulder3, origin xyz=0 -0.1115 0 rpy=0 0 0
- added joint jtoe0: type fixed, parent lower0, child toe0, origin xyz=0 0 -0.213 rpy=0 0 0
- added joint jtoe1: type fixed, parent lower1, child toe1, origin xyz=0 0 -0.213 rpy=0 0 0
- added joint jtoe2: type fixed, parent lower2, child toe2, origin xyz=0 0 -0.213 rpy=0 0 0
- added joint jtoe3: type fixed, parent lower3, child toe3, origin xyz=0 0 -0.213 rpy=0 0 0
- joint floating_base: parent base -> body
