Commit message: modified all xacros

File: quad_simulator/a1_description/xacro/gazebo.xacro (robot description, xacro)
@@ -59,40 +59,4 @@
     </gazebo>
     <!-- Foot contacts. -->
-    <!-- <gazebo reference="lower0">
-        <sensor name="FR_foot_contact" type="contact">
-        <update_rate>100</update_rate>
-        <plugin name="contactPlugin" filename="libunitreeFootContactPlugin.so"/>
-        <contact>
-            <collision>FR_calf_fixed_joint_lump__FR_foot_collision_1</collision>
-        </contact>
-        </sensor>
-    </gazebo>
-    <gazebo reference="lower1">
-        <sensor name="FL_foot_contact" type="contact">
-        <update_rate>100</update_rate>
-        <plugin name="contactPlugin" filename="libunitreeFootContactPlugin.so"/>
-        <contact>
-            <collision>FL_calf_fixed_joint_lump__FL_foot_collision_1</collision>
-        </contact>
-        </sensor>
-    </gazebo>
-    <gazebo reference="lower2">
-        <sensor name="RR_foot_contact" type="contact">
-        <update_rate>100</update_rate>
-        <plugin name="contactPlugin" filename="libunitreeFootContactPlugin.so"/>
-        <contact>
-            <collision>RR_calf_fixed_joint_lump__RR_foot_collision_1</collision>
-        </contact>
-        </sensor>
-    </gazebo>
-    <gazebo reference="lower3">
-        <sensor name="RL_foot_contact" type="contact">
-        <update_rate>100</update_rate>
-        <plugin name="contactPlugin" filename="libunitreeFootContactPlugin.so"/>
-        <contact>
-            <collision>RL_calf_fixed_joint_lump__RL_foot_collision_1</collision>
-        </contact>
-        </sensor>
-    </gazebo> -->
     <gazebo reference="toe0">
         <sensor name="toe0_contact" type="contact">

File: quad_simulator/go2_description/xacro/gazebo.xacro (robot description, xacro)
@@ -7,4 +7,7 @@
             <robotSimType>gazebo_ros_control/DefaultRobotHWSim</robotSimType>
         </plugin>
+        <plugin filename="libground_truth_estimator.so" name="ground_truth_estimator">
+            <updateRateHZ>500.0</updateRateHZ>
+        </plugin>
     </gazebo>
     <!-- Show the trajectory of trunk center. -->
@@ -13,5 +16,5 @@
             <frequency>10</frequency>
             <plot>
-                <link>base</link>
+                <link>body</link>
                 <pose>0 0 0 0 0 0</pose>
                 <material>Gazebo/Yellow</material>
@@ -55,42 +58,62 @@
     </gazebo>
     <!-- Foot contacts. -->
-    <gazebo reference="FR_calf">
-        <sensor name="FR_foot_contact" type="contact">
-        <update_rate>100</update_rate>
-        <plugin name="contactPlugin" filename="libunitreeFootContactPlugin.so"/>
-        <contact>
-            <collision>FR_calf_fixed_joint_lump__FR_foot_collision_1</collision>
-        </contact>
-        </sensor>
-    </gazebo>
-    <gazebo reference="FL_calf">
-        <sensor name="FL_foot_contact" type="contact">
-        <update_rate>100</update_rate>
-        <plugin name="contactPlugin" filename="libunitreeFootContactPlugin.so"/>
-        <contact>
-            <collision>FL_calf_fixed_joint_lump__FL_foot_collision_1</collision>
-        </contact>
-        </sensor>
-    </gazebo>
-    <gazebo reference="RR_calf">
-        <sensor name="RR_foot_contact" type="contact">
-        <update_rate>100</update_rate>
-        <plugin name="contactPlugin" filename="libunitreeFootContactPlugin.so"/>
-        <contact>
-            <collision>RR_calf_fixed_joint_lump__RR_foot_collision_1</collision>
-        </contact>
-        </sensor>
-    </gazebo>
-    <gazebo reference="RL_calf">
-        <sensor name="RL_foot_contact" type="contact">
-        <update_rate>100</update_rate>
-        <plugin name="contactPlugin" filename="libunitreeFootContactPlugin.so"/>
-        <contact>
-            <collision>RL_calf_fixed_joint_lump__RL_foot_collision_1</collision>
-        </contact>
+    <gazebo reference="toe0">
+        <sensor name="toe0_contact" type="contact">
+            <plugin name="toe0_plugin" filename="libgazebo_ros_bumper.so">
+                <alwaysOn>true</alwaysOn>
+                <updateRate>500</updateRate>
+                <bumperTopicName>gazebo/toe0_contact_state</bumperTopicName>
+                <frameName>world</frameName>
+            </plugin>
+            <contact>
+                <collision>toe0_collision</collision>
+            </contact>
+            <update_rate>500</update_rate>
+        </sensor>
+    </gazebo>
+    <gazebo reference="toe1">
+        <sensor name="toe1_contact" type="contact">
+            <plugin name="toe1_plugin" filename="libgazebo_ros_bumper.so">
+                <alwaysOn>true</alwaysOn>
+                <updateRate>500</updateRate>
+                <bumperTopicName>gazebo/toe1_contact_state</bumperTopicName>
+                <frameName>world</frameName>
+            </plugin>
+            <contact>
+                <collision>toe1_collision</collision>
+            </contact>
+            <update_rate>500</update_rate>
+        </sensor>
+    </gazebo>
+    <gazebo reference="toe2">
+        <sensor name="toe2_contact" type="contact">
+            <plugin name="toe2_plugin" filename="libgazebo_ros_bumper.so">
+                <alwaysOn>true</alwaysOn>
+                <updateRate>500</updateRate>
+                <bumperTopicName>gazebo/toe2_contact_state</bumperTopicName>
+                <frameName>world</frameName>
+            </plugin>
+            <contact>
+                <collision>toe2_collision</collision>
+            </contact>
+            <update_rate>500</update_rate>
+        </sensor>
+    </gazebo>
+    <gazebo reference="toe3">
+        <sensor name="toe3_contact" type="contact">
+            <plugin name="toe3_plugin" filename="libgazebo_ros_bumper.so">
+                <alwaysOn>true</alwaysOn>
+                <updateRate>500</updateRate>
+                <bumperTopicName>gazebo/toe3_contact_state</bumperTopicName>
+                <frameName>world</frameName>
+            </plugin>
+            <contact>
+                <collision>toe3_collision</collision>
+            </contact>
+            <update_rate>500</update_rate>
         </sensor>
     </gazebo>
     <!-- Visualization of Foot contacts. -->
-    <gazebo reference="FR_foot">
+    <!-- <gazebo reference="FR_foot">
         <visual>
             <plugin name="drawForcePlugin" filename="libunitreeDrawForcePlugin.so">
@@ -119,6 +142,6 @@
             </plugin>
         </visual>
-    </gazebo>
-    <gazebo reference="base">
+    </gazebo> -->
+    <gazebo reference="body">
         <turnGravityOff>false</turnGravityOff>
     </gazebo>
@@ -138,96 +161,96 @@
     </gazebo>
     <!-- FL leg -->
-    <gazebo reference="FL_hip">
-        <mu1>0.2</mu1>
-        <mu2>0.2</mu2>
-    </gazebo>
-    <gazebo reference="FL_thigh">
-        <mu1>0.2</mu1>
-        <mu2>0.2</mu2>
-        <self_collide>1</self_collide>
-        <kp  value="1000000.0"/>
-        <kd  value="1.0"/>
-    </gazebo>
-    <gazebo reference="FL_calf">
-        <mu1>0.2</mu1>
-        <mu2>0.2</mu2>
-        <self_collide>1</self_collide>
-    </gazebo>
-    <gazebo reference="FL_foot">
-        <mu1>0.6</mu1>
-        <mu2>0.6</mu2>
-        <self_collide>1</self_collide>
+    <gazebo reference="hip0">
+        <mu1>0.2</mu1>
+        <mu2>0.2</mu2>
+    </gazebo>
+    <gazebo reference="upper0">
+        <mu1>0.2</mu1>
+        <mu2>0.2</mu2>
+        <self_collide>0</self_collide>
+        <kp  value="1000000.0"/>
+        <kd  value="1.0"/>
+    </gazebo>
+    <gazebo reference="lower0">
+        <mu1>0.2</mu1>
+        <mu2>0.2</mu2>
+        <self_collide>0</self_collide>
+    </gazebo>
+    <gazebo reference="toe0">
+        <mu1>0.6</mu1>
+        <mu2>0.6</mu2>
+        <self_collide>0</self_collide>
+        <kp  value="1000000.0"/>
+        <kd  value="1.0"/>
+    </gazebo>
+    <!-- RL leg -->
+    <gazebo reference="hip1">
+        <mu1>0.2</mu1>
+        <mu2>0.2</mu2>
+    </gazebo>
+    <gazebo reference="upper1">
+        <mu1>0.2</mu1>
+        <mu2>0.2</mu2>
+        <self_collide>0</self_collide>
+        <kp  value="1000000.0"/>
+        <kd  value="1.0"/>
+    </gazebo>
+    <gazebo reference="lower1">
+        <mu1>0.2</mu1>
+        <mu2>0.2</mu2>
+        <self_collide>0</self_collide>
+    </gazebo>
+    <gazebo reference="toe1">
+        <mu1>0.6</mu1>
+        <mu2>0.6</mu2>
+        <self_collide>0</self_collide>
         <kp  value="1000000.0"/>
         <kd  value="1.0"/>
     </gazebo>
     <!-- FR leg -->
-    <gazebo reference="FR_hip">
-        <mu1>0.2</mu1>
-        <mu2>0.2</mu2>
-    </gazebo>
-    <gazebo reference="FR_thigh">
-        <mu1>0.2</mu1>
-        <mu2>0.2</mu2>
-        <self_collide>1</self_collide>
-        <kp  value="1000000.0"/>
-        <kd  value="1.0"/>
-    </gazebo>
-    <gazebo reference="FR_calf">
-        <mu1>0.2</mu1>
-        <mu2>0.2</mu2>
-        <self_collide>1</self_collide>
-    </gazebo>
-    <gazebo reference="FR_foot">
-        <mu1>0.6</mu1>
-        <mu2>0.6</mu2>
-        <self_collide>1</self_collide>
-        <kp  value="1000000.0"/>
-        <kd  value="1.0"/>
-    </gazebo>
-    <!-- RL leg -->
-    <gazebo reference="RL_hip">
-        <mu1>0.2</mu1>
-        <mu2>0.2</mu2>
-    </gazebo>
-    <gazebo reference="RL_thigh">
-        <mu1>0.2</mu1>
-        <mu2>0.2</mu2>
-        <self_collide>1</self_collide>
-        <kp  value="1000000.0"/>
-        <kd  value="1.0"/>
-    </gazebo>
-    <gazebo reference="RL_calf">
-        <mu1>0.2</mu1>
-        <mu2>0.2</mu2>
-        <self_collide>1</self_collide>
-    </gazebo>
-    <gazebo reference="RL_foot">
-        <mu1>0.6</mu1>
-        <mu2>0.6</mu2>
-        <self_collide>1</self_collide>
+    <gazebo reference="hip2">
+        <mu1>0.2</mu1>
+        <mu2>0.2</mu2>
+    </gazebo>
+    <gazebo reference="upper2">
+        <mu1>0.2</mu1>
+        <mu2>0.2</mu2>
+        <self_collide>0</self_collide>
+        <kp  value="1000000.0"/>
+        <kd  value="1.0"/>
+    </gazebo>
+    <gazebo reference="lower2">
+        <mu1>0.2</mu1>
+        <mu2>0.2</mu2>
+        <self_collide>0</self_collide>
+    </gazebo>
+    <gazebo reference="toe2">
+        <mu1>0.6</mu1>
+        <mu2>0.6</mu2>
+        <self_collide>0</self_collide>
         <kp  value="1000000.0"/>
         <kd  value="1.0"/>
     </gazebo>
     <!-- RR leg -->
-    <gazebo reference="RR_hip">
-        <mu1>0.2</mu1>
-        <mu2>0.2</mu2>
-    </gazebo>
-    <gazebo reference="RR_thigh">
-        <mu1>0.2</mu1>
-        <mu2>0.2</mu2>
-        <self_collide>1</self_collide>
-        <kp  value="1000000.0"/>
-        <kd  value="1.0"/>
-    </gazebo>
-    <gazebo reference="RR_calf">
-        <mu1>0.2</mu1>
-        <mu2>0.2</mu2>
-        <self_collide>1</self_collide>
-    </gazebo>
-    <gazebo reference="RR_foot">
-        <mu1>0.6</mu1>
-        <mu2>0.6</mu2>
-        <self_collide>1</self_collide>
+    <gazebo reference="hip3">
+        <mu1>0.2</mu1>
+        <mu2>0.2</mu2>
+    </gazebo>
+    <gazebo reference="upper3">
+        <mu1>0.2</mu1>
+        <mu2>0.2</mu2>
+        <self_collide>0</self_collide>
+        <kp  value="1000000.0"/>
+        <kd  value="1.0"/>
+    </gazebo>
+    <gazebo reference="lower3">
+        <mu1>0.2</mu1>
+        <mu2>0.2</mu2>
+        <self_collide>0</self_collide>
+    </gazebo>
+    <gazebo reference="toe3">
+        <mu1>0.6</mu1>
+        <mu2>0.6</mu2>
+        <self_collide>0</self_collide>
         <kp  value="1000000.0"/>
         <kd  value="1.0"/>

File: quad_simulator/go2_description/xacro/robot.xacro (robot description, xacro)
@@ -109,5 +109,5 @@
         </collision>
     </link>
-        <!--FL-->
+    <!--FL-->
     <xacro:leg suffix="0" mirror="1" mirror_dae="True" front_hind="1" front_hind_dae="True"
                hipJointName="0" kneeJointName="1" abductionJointName="8">

Commit message: getting error while launching gazebo

File: quad_simulator/a1_description/xacro/gazebo.xacro (robot description, xacro)
@@ -115,33 +115,4 @@
         </sensor>
     </gazebo>
-    <!-- Visualization of Foot contacts. -->
-    <!-- <gazebo reference="toe0">
-        <visual>
-            <plugin name="drawForcePlugin" filename="libunitreeDrawForcePlugin.so">
-                <topicName>FR_foot_contact</topicName>
-            </plugin>
-        </visual>
-    </gazebo>
-    <gazebo reference="toe1">
-        <visual>
-            <plugin name="drawForcePlugin" filename="libunitreeDrawForcePlugin.so">
-                <topicName>FL_foot_contact</topicName>
-            </plugin>
-        </visual>
-    </gazebo>
-    <gazebo reference="toe2">
-        <visual>
-            <plugin name="drawForcePlugin" filename="libunitreeDrawForcePlugin.so">
-                <topicName>RR_foot_contact</topicName>
-            </plugin>
-        </visual>
-    </gazebo>
-    <gazebo reference="toe3">
-        <visual>
-            <plugin name="drawForcePlugin" filename="libunitreeDrawForcePlugin.so">
-                <topicName>RL_foot_contact</topicName>
-            </plugin>
-        </visual>
-    </gazebo> -->
     <gazebo reference="body">
         <material>Gazebo/Green</material>

File: quad_simulator/go2_description/xacro/gazebo.xacro (robot description, xacro)
@@ -115,32 +115,4 @@
     </gazebo>
     <!-- Visualization of Foot contacts. -->
-    <!-- <gazebo reference="FR_foot">
-        <visual>
-            <plugin name="drawForcePlugin" filename="libunitreeDrawForcePlugin.so">
-                <topicName>FR_foot_contact</topicName>
-            </plugin>
-        </visual>
-    </gazebo>
-    <gazebo reference="FL_foot">
-        <visual>
-            <plugin name="drawForcePlugin" filename="libunitreeDrawForcePlugin.so">
-                <topicName>FL_foot_contact</topicName>
-            </plugin>
-        </visual>
-    </gazebo>
-    <gazebo reference="RR_foot">
-        <visual>
-            <plugin name="drawForcePlugin" filename="libunitreeDrawForcePlugin.so">
-                <topicName>RR_foot_contact</topicName>
-            </plugin>
-        </visual>
-    </gazebo>
-    <gazebo reference="RL_foot">
-        <visual>
-            <plugin name="drawForcePlugin" filename="libunitreeDrawForcePlugin.so">
-                <topicName>RL_foot_contact</topicName>
-            </plugin>
-        </visual>
-    </gazebo> -->
     <gazebo reference="body">
         <turnGravityOff>false</turnGravityOff>

Commit message: still trying to fix gz error

File: quad_simulator/a1_description/xacro/gazebo.xacro (robot description, xacro)
@@ -11,26 +11,4 @@
         </plugin>
     </gazebo>
-    <!-- Show the trajectory of trunk center. -->
-    <!-- <gazebo>
-        <plugin name="3dplot" filename="libLinkPlot3DPlugin.so">
-            <frequency>10</frequency>
-            <plot>
-                <link>body</link>
-                <pose>0 0 0 0 0 0</pose>
-                <material>Gazebo/Yellow</material>
-            </plot>
-        </plugin>
-    </gazebo> -->
-    <!-- Show the trajectory of foot. You can add another trajectory about another foot. -->
-    <!-- <gazebo>
-        <plugin name="3dplot" filename="libLinkPlot3DPlugin.so">
-            <frequency>100</frequency>
-            <plot>
-                <link>FL_foot</link>
-                <pose>0 0 0 0 0 0</pose>
-                <material>Gazebo/Green</material>
-            </plot>
-        </plugin>
-    </gazebo> -->
     <gazebo>
         <plugin filename="libgazebo_ros_force.so" name="gazebo_ros_force">

File: quad_simulator/go2_description/xacro/gazebo.xacro (robot description, xacro)
@@ -23,5 +23,5 @@
     </gazebo-->
     <!-- Show the trajectory of foot. You can add another trajectory about another foot. -->
-     <gazebo>
+     <!-- <gazebo>
         <plugin name="3dplot" filename="libLinkPlot3DPlugin.so">
             <frequency>100</frequency>
@@ -31,5 +31,5 @@
             </plot>
         </plugin>
-    </gazebo>
+    </gazebo> -->
     <gazebo>
         <plugin filename="libgazebo_ros_force.so" name="gazebo_ros_force">
